File: propagation_delay_led_pulser.kicad_pcb (KiCad board)
At the start: 2 copper layers, 33 x 48 mm, 15 parts, among them J1 Power/Bias In, J2 Pulse Out, U1 74AC14, U2 ICM7555xB, U3 74AHC1G00

Commit message: Removed extra vias and changed 0612 caps to 1206
  should ease soldering greatly
  Hopefully all done for v1.1
Parts:
- C1: footprint Resistor_SMD:R_1206_3216Metric_Pad1.30x1.75mm_HandSolder -> Capacitor_SMD:C_1206_3216Metric_Pad1.33x1.80mm_HandSolder
- C3, C4, C5, C6: footprint Resistor_SMD:R_0612_1632Metric_Pad1.18x3.40mm_HandSolder -> Capacitor_SMD:C_1206_3216Metric_Pad1.33x1.80mm_HandSolder
- moved C4 0.70 mm to (214.4, 69.8), turned to 0 degrees
- moved C3 0.64 mm to (208.8, 63.9)
Routing:
- net GND: track 48.3 -> 18.0 mm, vias 27 -> 11
- net VCC: track 66.5 -> 63.1 mm
- net /Inv3toNand: track 14.1 -> 15.0 mm
- net /Pulser_out: track 32.8 -> 32.3 mm
Other:
- board text added: "Propagation Delay LED Pulser HugonLabs 2022-04-12 V1.1"
- board text added: "V1.1 2022-04-12"
- board text removed: "Propagation Delay LED Pulser HugonLabs 2022-02-28 V1"
- board text removed: "V1 2022-02-28"
